File: StepperServo.sch (KiCad schematic (older format))
At the start: 23 parts, among them J1 Input, J2 Microstep, J3 Stepper, J4 Servo1, J5 Servo2, Q1 ZVNL110A, Q2 ZVNL110A, U1 ATtiny84-20PU

Commit message: Updated schematic
Parts:
- TP7: value TestPoint -> ~FLT
- U1: symbol MCU_Microchip_ATtiny:ATtiny84-20PU -> StepperServo-rescue:ATtiny84-20PU-MCU_Microchip_ATtiny
Other:
- moved on the sheet: C3, TP7
Changed lines of the file:
@@
 EESchema Schematic File Version 4
-EELAYER 29 0
+EELAYER 30 0
 EELAYER END
 $Descr USLetter 11000 8500
@@
 $EndComp
 $Comp
-L MCU_Microchip_ATtiny:ATtiny84-20PU U1
+L StepperServo-rescue:ATtiny84-20PU-MCU_Microchip_ATtiny U1
 U 1 1 5E6C0AC4
 P 4350 2650
@@
 L Device:CP1 C3
 U 1 1 5E6C68A8
-P 8600 2050
-F 0 "C3" H 8715 2096 50  0000 L CNN
-F 1 "100uf" H 8715 2005 50  0000 L CNN
-F 2 "" H 8600 2050 50  0001 C CNN
-F 3 "~" H 8600 2050 50  0001 C CNN
-	1    8600 2050
-	1    0    0    -1
-$EndComp
-Wire Wire Line
-	8600 2200 8600 3550
-Wire Wire Line
-	8600 3550 8350 3550
+P 8700 2050
+F 0 "C3" H 8815 2096 50  0000 L CNN
+F 1 "100uf" H 8815 2005 50  0000 L CNN
+F 2 "" H 8700 2050 50  0001 C CNN
+F 3 "~" H 8700 2050 50  0001 C CNN
+	1    8700 2050
+	1    0    0    -1
+$EndComp
+Wire Wire Line
+	8700 2200 8700 3550
+Wire Wire Line
+	8700 3550 8350 3550
 Wire Wire Line
 	8150 3550 8150 3450
@@
 L power:+12V #PWR010
 U 1 1 5E6C9B61
-P 8300 1750
-F 0 "#PWR010" H 8300 1600 50  0001 C CNN
-F 1 "+12V" H 8315 1923 50  0000 C CNN
-F 2 "" H 8300 1750 50  0001 C CNN
-F 3 "" H 8300 1750 50  0001 C CNN
-	1    8300 1750
+P 8300 1650
+F 0 "#PWR010" H 8300 1500 50  0001 C CNN
+F 1 "+12V" H 8315 1823 50  0000 C CNN
+F 2 "" H 8300 1650 50  0001 C CNN
+F 3 "" H 8300 1650 50  0001 C CNN
+	1    8300 1650
 	1    0    0    -1
 $EndComp
@@
 $EndComp
 Wire Wire Line
-	2850 2850 2850 3550
-Wire Wire Line
-	2850 3550 4350 3550
-Wire Wire Line
-	2850 2550 2850 1750
-Wire Wire Line
-	2850 1750 4350 1750
+	2850 2850 2850 3650
 $Comp
 L power:+5V #PWR08
 U 1 1 5E6CC787
-P 4350 1750
-F 0 "#PWR08" H 4350 1600 50  0001 C CNN
-F 1 "+5V" H 4365 1923 50  0000 C CNN
-F 2 "" H 4350 1750 50  0001 C CNN
-F 3 "" H 4350 1750 50  0001 C CNN
-	1    4350 1750
-	1    0    0    -1
-$EndComp
-Connection ~ 4350 1750
+P 4350 1650
+F 0 "#PWR08" H 4350 1500 50  0001 C CNN
+F 1 "+5V" H 4365 1823 50  0000 C CNN
+F 2 "" H 4350 1650 50  0001 C CNN
+F 3 "" H 4350 1650 50  0001 C CNN
+	1    4350 1650
+	1    0    0    -1
+$EndComp
 $Comp
 L power:GND #PWR09
 U 1 1 5E6CC967
-P 4350 3550
-F 0 "#PWR09" H 4350 3300 50  0001 C CNN
-F 1 "GND" H 4355 3377 50  0000 C CNN
-F 2 "" H 4350 3550 50  0001 C CNN
-F 3 "" H 4350 3550 50  0001 C CNN
-	1    4350 3550
-	1    0    0    -1
-$EndComp
-Connection ~ 4350 3550
+P 4350 3650
+F 0 "#PWR09" H 4350 3400 50  0001 C CNN
+F 1 "GND" H 4355 3477 50  0000 C CNN
+F 2 "" H 4350 3650 50  0001 C CNN
+F 3 "" H 4350 3650 50  0001 C CNN
+	1    4350 3650
+	1    0    0    -1
+$EndComp
 Wire Wire Line
 	1500 2750 1950 2750
@@
 	1950 2750 1950 2850
 Wire Wire Line
-	1950 3550 2850 3550
-Connection ~ 2850 3550
-Wire Wire Line
-	8600 1900 8600 1750
-Wire Wire Line
-	8600 1750 8300 1750
-Wire Wire Line
-	8050 2050 8050 1750
-Wire Wire Line
-	8050 1750 8300 1750
-Connection ~ 8300 1750
+	1950 3650 2850 3650
+Wire Wire Line
+	8700 1900 8700 1650
+Wire Wire Line
+	8700 1650 8300 1650
+Wire Wire Line
+	8050 2050 8050 1650
+Wire Wire Line
+	8050 1650 8300 1650
+Connection ~ 8300 1650
 $Comp
 L StepperServo:ZVNL110A Q2
@@
 Connection ~ 1950 2850
 Wire Wire Line
-	1950 2850 1950 3550
+	1950 2850 1950 3650
 Wire Wire Line
 	1950 2550 1950 2350
@@
 	7400 2450 7400 2350
 Wire Wire Line
-	7400 1750 4350 1750
-Wire Wire Line
 	7650 2350 7400 2350
 Connection ~ 7400 2350
 Wire Wire Line
-	7400 2350 7400 1750
-Wire Wire Line
 	7650 2650 6900 2650
 Wire Wire Line
@@
 L Connector:TestPoint TP7
 U 1 1 5E76150C
-P 7500 1750
-F 0 "TP7" H 7558 1868 50  0000 L CNN
-F 1 "TestPoint" H 7558 1777 50  0000 L CNN
-F 2 "" H 7700 1750 50  0001 C CNN
-F 3 "~" H 7700 1750 50  0001 C CNN
-	1    7500 1750
-	1    0    0    -1
-$EndComp
-Wire Wire Line
-	7500 1750 7500 2250
+P 7500 1650
+F 0 "TP7" H 7558 1768 50  0000 L CNN
+F 1 "~FLT" H 7558 1677 50  0000 L CNN
+F 2 "" H 7700 1650 50  0001 C CNN
+F 3 "~" H 7700 1650 50  0001 C CNN
+	1    7500 1650
+	1    0    0    -1
+$EndComp
+Wire Wire Line
+	7500 1650 7500 2250
 Wire Wire Line
 	7500 2250 7650 2250
@@
 Wire Wire Line
 	5050 2250 4950 2250
+Wire Wire Line
+	4350 1750 4350 1650
+Wire Wire Line
+	4350 1650 2850 1650
+Wire Wire Line
+	2850 1650 2850 2550
+Connection ~ 4350 1650
+Wire Wire Line
+	7400 1650 4350 1650
+Wire Wire Line
+	7400 1650 7400 2350
+Wire Wire Line
+	4350 3650 4350 3550
+Wire Wire Line
+	4350 3650 2850 3650
+Connection ~ 4350 3650
+Connection ~ 2850 3650
 $EndSCHEMATC

Commit message: Fixed tantalum and assigned footprints
Parts:
- C1: footprint (none) -> Capacitor_THT:CP_Radial_Tantal_D6.0mm_P2.50mm; symbol Device:C -> Device:CP1
- C2: footprint (none) -> Capacitor_THT:C_Disc_D5.0mm_W2.5mm_P2.50mm
- C3: footprint (none) -> Capacitor_THT:CP_Radial_D5.0mm_P2.50mm
- J1: footprint (none) -> Connector_PinHeader_2.54mm:PinHeader_1x06_P2.54mm_Vertical
- J2: footprint (none) -> Connector_PinHeader_1.27mm:PinHeader_2x03_P1.27mm_Vertical
- J3: footprint (none) -> Connector_PinHeader_2.54mm:PinHeader_1x04_P2.54mm_Vertical
- J4, J5: footprint (none) -> Connector_PinHeader_2.54mm:PinHeader_1x03_P2.54mm_Vertical
- R1, R2, R3, R4: footprint (none) -> Resistor_THT:R_Axial_DIN0207_L6.3mm_D2.5mm_P7.62mm_Horizontal
- TP1, TP2, TP3, TP4, TP5, TP6, TP7: footprint (none) -> TestPoint:TestPoint_Plated_Hole_D2.0mm
Changed lines of the file:
@@
 F 0 "C3" H 8815 2096 50  0000 L CNN
 F 1 "100uf" H 8815 2005 50  0000 L CNN
-F 2 "" H 8700 2050 50  0001 C CNN
+F 2 "Capacitor_THT:CP_Radial_D5.0mm_P2.50mm" H 8700 2050 50  0001 C CNN
 F 3 "~" H 8700 2050 50  0001 C CNN
 	1    8700 2050
@@
 $EndComp
 $Comp
-L Device:C C1
+L Device:CP1 C1
 U 1 1 5E6CAA08
 P 2100 2700
 F 0 "C1" H 2215 2746 50  0000 L CNN
 F 1 "10uf" H 2215 2655 50  0000 L CNN
-F 2 "" H 2138 2550 50  0001 C CNN
+F 2 "Capacitor_THT:CP_Radial_Tantal_D6.0mm_P2.50mm" H 2138 2550 50  0001 C CNN
 F 3 "~" H 2100 2700 50  0001 C CNN
 	1    2100 2700
@@
 F 0 "C2" H 2965 2746 50  0000 L CNN
 F 1 "0.1uf" H 2965 2655 50  0000 L CNN
-F 2 "" H 2888 2550 50  0001 C CNN
+F 2 "Capacitor_THT:C_Disc_D5.0mm_W2.5mm_P2.50mm" H 2888 2550 50  0001 C CNN
 F 3 "~" H 2850 2700 50  0001 C CNN
 	1    2850 2700
@@
 F 0 "R2" H 2170 4496 50  0000 L CNN
 F 1 "10K" H 2170 4405 50  0000 L CNN
-F 2 "" V 2030 4450 50  0001 C CNN
+F 2 "Resistor_THT:R_Axial_DIN0207_L6.3mm_D2.5mm_P7.62mm_Horizontal" V 2030 4450 50  0001 C CNN
 F 3 "~" H 2100 4450 50  0001 C CNN
 	1    2100 4450
@@
 F 0 "R4" H 2970 4496 50  0000 L CNN
 F 1 "10K" H 2970 4405 50  0000 L CNN
-F 2 "" V 2830 4450 50  0001 C CNN
+F 2 "Resistor_THT:R_Axial_DIN0207_L6.3mm_D2.5mm_P7.62mm_Horizontal" V 2830 4450 50  0001 C CNN
 F 3 "~" H 2900 4450 50  0001 C CNN
 	1    2900 4450
@@
 F 0 "R1" H 2120 5596 50  0000 L CNN
 F 1 "10K" H 2120 5505 50  0000 L CNN
-F 2 "" V 1980 5550 50  0001 C CNN
+F 2 "Resistor_THT:R_Axial_DIN0207_L6.3mm_D2.5mm_P7.62mm_Horizontal" V 1980 5550 50  0001 C CNN
 F 3 "~" H 2050 5550 50  0001 C CNN
 	1    2050 5550
@@
 F 0 "R3" H 2920 5596 50  0000 L CNN
 F 1 "10K" H 2920 5505 50  0000 L CNN
-F 2 "" V 2780 5550 50  0001 C CNN
+F 2 "Resistor_THT:R_Axial_DIN0207_L6.3mm_D2.5mm_P7.62mm_Horizontal" V 2780 5550 50  0001 C CNN
 F 3 "~" H 2850 5550 50  0001 C CNN
 	1    2850 5550
@@
 F 0 "J5" H 9380 5092 50  0000 L CNN
 F 1 "Servo2" H 9380 5001 50  0000 L CNN
-F 2 "" H 9300 5050 50  0001 C CNN
+F 2 "Connector_PinHeader_2.54mm:PinHeader_1x03_P2.54mm_Vertical" H 9300 5050 50  0001 C CNN
 F 3 "~" H 9300 5050 50  0001 C CNN
 	1    9300 5050
@@
 F 0 "J1" H 1218 3067 50  0000 C CNN
 F 1 "Input" H 1218 2976 50  0000 C CNN
-F 2 "" H 1300 2650 50  0001 C CNN
+F 2 "Connector_PinHeader_2.54mm:PinHeader_1x06_P2.54mm_Vertical" H 1300 2650 50  0001 C CNN
 F 3 "~" H 1300 2650 50  0001 C CNN
 	1    1300 2650
@@
 F 0 "J3" H 9380 2692 50  0000 L CNN
 F 1 "Stepper" H 9380 2601 50  0000 L CNN
-F 2 "" H 9300 2700 50  0001 C CNN
+F 2 "Connector_PinHeader_2.54mm:PinHeader_1x04_P2.54mm_Vertical" H 9300 2700 50  0001 C CNN
 F 3 "~" H 9300 2700 50  0001 C CNN
 	1    9300 2700
@@
 F 0 "J4" H 9380 4592 50  0000 L CNN
 F 1 "Servo1" H 9380 4501 50  0000 L CNN
-F 2 "" H 9300 4550 50  0001 C CNN
+F 2 "Connector_PinHeader_2.54mm:PinHeader_1x03_P2.54mm_Vertical" H 9300 4550 50  0001 C CNN
 F 3 "~" H 9300 4550 50  0001 C CNN
 	1    9300 4550
@@
 F 0 "J2" H 7150 3467 50  0000 C CNN
 F 1 "Microstep" H 7150 3376 50  0000 C CNN
-F 2 "" H 7100 3150 50  0001 C CNN
+F 2 "Connector_PinHeader_1.27mm:PinHeader_2x03_P1.27mm_Vertical" H 7100 3150 50  0001 C CNN
 F 3 "~" H 7100 3150 50  0001 C CNN
 	1    7100 3150
@@
 F 0 "TP7" H 7558 1768 50  0000 L CNN
 F 1 "~FLT" H 7558 1677 50  0000 L CNN
-F 2 "" H 7700 1650 50  0001 C CNN
+F 2 "TestPoint:TestPoint_Plated_Hole_D2.0mm" H 7700 1650 50  0001 C CNN
 F 3 "~" H 7700 1650 50  0001 C CNN
 	1    7500 1650
@@
 F 0 "TP1" V 5004 2438 50  0000 L CNN
 F 1 "PA2" V 5095 2438 50  0000 L CNN
-F 2 "" H 5250 2250 50  0001 C CNN
+F 2 "TestPoint:TestPoint_Plated_Hole_D2.0mm" H 5250 2250 50  0001 C CNN
 F 3 "~" H 5250 2250 50  0001 C CNN
 	1    5050 2250
@@
 F 0 "TP5" V 5304 2538 50  0000 L CNN
 F 1 "PA3" V 5395 2538 50  0000 L CNN
-F 2 "" H 5550 2350 50  0001 C CNN
+F 2 "TestPoint:TestPoint_Plated_Hole_D2.0mm" H 5550 2350 50  0001 C CNN
 F 3 "~" H 5550 2350 50  0001 C CNN
 	1    5350 2350
@@
 F 0 "TP2" V 5004 2738 50  0000 L CNN
 F 1 "PA5" V 5095 2738 50  0000 L CNN
-F 2 "" H 5250 2550 50  0001 C CNN
+F 2 "TestPoint:TestPoint_Plated_Hole_D2.0mm" H 5250 2550 50  0001 C CNN
 F 3 "~" H 5250 2550 50  0001 C CNN
 	1    5050 2550
@@
 F 0 "TP3" V 5004 2938 50  0000 L CNN
 F 1 "PA7" V 5095 2938 50  0000 L CNN
-F 2 "" H 5250 2750 50  0001 C CNN
+F 2 "TestPoint:TestPoint_Plated_Hole_D2.0mm" H 5250 2750 50  0001 C CNN
 F 3 "~" H 5250 2750 50  0001 C CNN
 	1    5050 2750
@@
 F 0 "TP4" V 5004 3338 50  0000 L CNN
 F 1 "PB2" V 5095 3338 50  0000 L CNN
-F 2 "" H 5250 3150 50  0001 C CNN
+F 2 "TestPoint:TestPoint_Plated_Hole_D2.0mm" H 5250 3150 50  0001 C CNN
 F 3 "~" H 5250 3150 50  0001 C CNN
 	1    5050 3150
@@
 F 0 "TP6" V 5304 3438 50  0000 L CNN
 F 1 "PB3" V 5395 3438 50  0000 L CNN
-F 2 "" H 5550 3250 50  0001 C CNN
+F 2 "TestPoint:TestPoint_Plated_Hole_D2.0mm" H 5550 3250 50  0001 C CNN
 F 3 "~" H 5550 3250 50  0001 C CNN
 	1    5350 3250

Commit message: PCB Layout
Parts:
- removed TP1: PA2, TestPoint:TestPoint_Plated_Hole_D2.0mm, symbol Connector:TestPoint
- removed TP2: PA5, TestPoint:TestPoint_Plated_Hole_D2.0mm, symbol Connector:TestPoint
- removed TP3: PA7, TestPoint:TestPoint_Plated_Hole_D2.0mm, symbol Connector:TestPoint
- removed TP4: PB2, TestPoint:TestPoint_Plated_Hole_D2.0mm, symbol Connector:TestPoint
- removed TP5: PA3, TestPoint:TestPoint_Plated_Hole_D2.0mm, symbol Connector:TestPoint
- removed TP6: PB3, TestPoint:TestPoint_Plated_Hole_D2.0mm, symbol Connector:TestPoint
- removed TP7: ~FLT, TestPoint:TestPoint_Plated_Hole_D2.0mm, symbol Connector:TestPoint
- J2: footprint Connector_PinHeader_1.27mm:PinHeader_2x03_P1.27mm_Vertical -> Connector_PinHeader_2.54mm:PinHeader_2x03_P2.54mm_Vertical; symbol Connector_Generic:Conn_02x03_Row_Letter_First -> Connector_Generic:Conn_02x03_Odd_Even
- R1, R2, R3, R4: footprint Resistor_THT:R_Axial_DIN0207_L6.3mm_D2.5mm_P7.62mm_Horizontal -> Resistor_THT:R_Axial_DIN0207_L6.3mm_D2.5mm_P2.54mm_Vertical
Connections:
- net GND: now also J2.1 (Pin_1), J2.3 (Pin_3), J2.5 (Pin_5); no longer J2.a1 (Pin_a1), J2.a2 (Pin_a2), J2.a3 (Pin_a3)
- net at A1.10 (M0): now also J2.2 (Pin_2); no longer J2.b1 (Pin_b1)
- net at A1.11 (M1): now also J2.4 (Pin_4); no longer J2.b2 (Pin_b2)
- net at A1.12 (M2): now also J2.6 (Pin_6); no longer J2.b3 (Pin_b3)
- no-connect marks 0 -> 7
Changed lines of the file:
@@
 F 0 "R2" H 2170 4496 50  0000 L CNN
 F 1 "10K" H 2170 4405 50  0000 L CNN
-F 2 "Resistor_THT:R_Axial_DIN0207_L6.3mm_D2.5mm_P7.62mm_Horizontal" V 2030 4450 50  0001 C CNN
+F 2 "Resistor_THT:R_Axial_DIN0207_L6.3mm_D2.5mm_P2.54mm_Vertical" V 2030 4450 50  0001 C CNN
 F 3 "~" H 2100 4450 50  0001 C CNN
 	1    2100 4450
@@
 F 0 "R4" H 2970 4496 50  0000 L CNN
 F 1 "10K" H 2970 4405 50  0000 L CNN
-F 2 "Resistor_THT:R_Axial_DIN0207_L6.3mm_D2.5mm_P7.62mm_Horizontal" V 2830 4450 50  0001 C CNN
+F 2 "Resistor_THT:R_Axial_DIN0207_L6.3mm_D2.5mm_P2.54mm_Vertical" V 2830 4450 50  0001 C CNN
 F 3 "~" H 2900 4450 50  0001 C CNN
 	1    2900 4450
@@
 F 0 "R1" H 2120 5596 50  0000 L CNN
 F 1 "10K" H 2120 5505 50  0000 L CNN
-F 2 "Resistor_THT:R_Axial_DIN0207_L6.3mm_D2.5mm_P7.62mm_Horizontal" V 1980 5550 50  0001 C CNN
+F 2 "Resistor_THT:R_Axial_DIN0207_L6.3mm_D2.5mm_P2.54mm_Vertical" V 1980 5550 50  0001 C CNN
 F 3 "~" H 2050 5550 50  0001 C CNN
 	1    2050 5550
@@
 F 0 "R3" H 2920 5596 50  0000 L CNN
 F 1 "10K" H 2920 5505 50  0000 L CNN
-F 2 "Resistor_THT:R_Axial_DIN0207_L6.3mm_D2.5mm_P7.62mm_Horizontal" V 2780 5550 50  0001 C CNN
+F 2 "Resistor_THT:R_Axial_DIN0207_L6.3mm_D2.5mm_P2.54mm_Vertical" V 2780 5550 50  0001 C CNN
 F 3 "~" H 2850 5550 50  0001 C CNN
 	1    2850 5550
@@
 	6600 4450 9100 4450
 $Comp
-L Connector_Generic:Conn_02x03_Row_Letter_First J2
+L Connector_Generic:Conn_02x03_Odd_Even J2
 U 1 1 5E716C25
 P 7100 3150
 F 0 "J2" H 7150 3467 50  0000 C CNN
 F 1 "Microstep" H 7150 3376 50  0000 C CNN
-F 2 "Connector_PinHeader_1.27mm:PinHeader_2x03_P1.27mm_Vertical" H 7100 3150 50  0001 C CNN
+F 2 "Connector_PinHeader_2.54mm:PinHeader_2x03_P2.54mm_Vertical" H 7100 3150 50  0001 C CNN
 F 3 "~" H 7100 3150 50  0001 C CNN
 	1    7100 3150
@@
 	6900 2650 6900 3050
 Connection ~ 6900 3050
-$Comp
-L Connector:TestPoint TP7
-U 1 1 5E76150C
-P 7500 1650
-F 0 "TP7" H 7558 1768 50  0000 L CNN
-F 1 "~FLT" H 7558 1677 50  0000 L CNN
-F 2 "TestPoint:TestPoint_Plated_Hole_D2.0mm" H 7700 1650 50  0001 C CNN
-F 3 "~" H 7700 1650 50  0001 C CNN
-	1    7500 1650
-	1    0    0    -1
-$EndComp
-Wire Wire Line
-	7500 1650 7500 2250
-Wire Wire Line
-	7500 2250 7650 2250
-$Comp
-L Connector:TestPoint TP1
-U 1 1 5E768EE0
-P 5050 2250
-F 0 "TP1" V 5004 2438 50  0000 L CNN
-F 1 "PA2" V 5095 2438 50  0000 L CNN
-F 2 "TestPoint:TestPoint_Plated_Hole_D2.0mm" H 5250 2250 50  0001 C CNN
-F 3 "~" H 5250 2250 50  0001 C CNN
-	1    5050 2250
-	0    1    1    0
-$EndComp
-$Comp
-L Connector:TestPoint TP5
-U 1 1 5E76A93A
-P 5350 2350
-F 0 "TP5" V 5304 2538 50  0000 L CNN
-F 1 "PA3" V 5395 2538 50  0000 L CNN
-F 2 "TestPoint:TestPoint_Plated_Hole_D2.0mm" H 5550 2350 50  0001 C CNN
-F 3 "~" H 5550 2350 50  0001 C CNN
-	1    5350 2350
-	0    1    1    0
-$EndComp
-$Comp
-L Connector:TestPoint TP2
-U 1 1 5E78DF8E
-P 5050 2550
-F 0 "TP2" V 5004 2738 50  0000 L CNN
-F 1 "PA5" V 5095 2738 50  0000 L CNN
-F 2 "TestPoint:TestPoint_Plated_Hole_D2.0mm" H 5250 2550 50  0001 C CNN
-F 3 "~" H 5250 2550 50  0001 C CNN
-	1    5050 2550
-	0    1    1    0
-$EndComp
-$Comp
-L Connector:TestPoint TP3
-U 1 1 5E78E3A2
-P 5050 2750
-F 0 "TP3" V 5004 2938 50  0000 L CNN
-F 1 "PA7" V 5095 2938 50  0000 L CNN
-F 2 "TestPoint:TestPoint_Plated_Hole_D2.0mm" H 5250 2750 50  0001 C CNN
-F 3 "~" H 5250 2750 50  0001 C CNN
-	1    5050 2750
-	0    1    1    0
-$EndComp
-$Comp
-L Connector:TestPoint TP4
-U 1 1 5E791778
-P 5050 3150
-F 0 "TP4" V 5004 3338 50  0000 L CNN
-F 1 "PB2" V 5095 3338 50  0000 L CNN
-F 2 "TestPoint:TestPoint_Plated_Hole_D2.0mm" H 5250 3150 50  0001 C CNN
-F 3 "~" H 5250 3150 50  0001 C CNN
-	1    5050 3150
-	0    1    1    0
-$EndComp
-$Comp
-L Connector:TestPoint TP6
-U 1 1 5E791B08
-P 5350 3250
-F 0 "TP6" V 5304 3438 50  0000 L CNN
-F 1 "PB3" V 5395 3438 50  0000 L CNN
-F 2 "TestPoint:TestPoint_Plated_Hole_D2.0mm" H 5550 3250 50  0001 C CNN
-F 3 "~" H 5550 3250 50  0001 C CNN
-	1    5350 3250
-	0    1    1    0
-$EndComp
-Wire Wire Line
-	5350 3250 4950 3250
-Wire Wire Line
-	5050 3150 4950 3150
-Wire Wire Line
-	5050 2750 4950 2750
-Wire Wire Line
-	5050 2550 4950 2550
-Wire Wire Line
-	5350 2350 4950 2350
-Wire Wire Line
-	5050 2250 4950 2250
 Wire Wire Line
 	4350 1750 4350 1650
@@
 Connection ~ 4350 3650
 Connection ~ 2850 3650
+NoConn ~ 7650 2250
+NoConn ~ 4950 2750
+NoConn ~ 4950 2550
+NoConn ~ 4950 2350
+NoConn ~ 4950 2250
+NoConn ~ 4950 3150
+NoConn ~ 4950 3250
 $EndSCHEMATC
